Commit message: python3対応

File: template.xacro (robot description, xacro)
@@ -21,5 +21,5 @@
       <origin rpy="{{sample.link_rpy}}" xyz="{{sample.link_xyz}}"/>
       <geometry>
-        <{{sample.link_size}}/>
+        <box size="{{sample.link_size}}"/>
       </geometry>
     </collision>
@@ -27,5 +27,5 @@
       <origin rpy="{{sample.link_rpy}}" xyz="{{sample.link_xyz}}"/>
       <geometry>
-        <{{sample.link_size}}/>
+        <box size="{{sample.link_size}}"/>
       </geometry>
       <material name="{{sample.link_color}}"/>

File: template_gazebo.xacro (robot description, xacro)
@@ -21,5 +21,5 @@
       <origin rpy="{{sample.link_rpy}}" xyz="{{sample.link_xyz}}"/>
       <geometry>
-        <{{sample.link_size}}/>
+        <box size="{{sample.link_size}}"/>
       </geometry>
     </collision>
@@ -27,5 +27,5 @@
       <origin rpy="{{sample.link_rpy}}" xyz="{{sample.link_xyz}}"/>
       <geometry>
-        <{{sample.link_size}}/>
+        <box size="{{sample.link_size}}"/>
       </geometry>
       <material name="{{sample.link_color}}"/>
